Commit message: New Model made by jiyong

File: urdf/SUBO3.urdf (robot description, URDF)
Before this commit: robot SUBO3, 21 links, 20 joints
Links:
- link L_ANKLE_PITCH_LINK: mass 1.23810021571121 -> 0.841930312664941
- link L_ANKLE_ROLL_LINK: mass 0.274125500095123 -> 0.274125500097104
- link L_FOOTPAD_LINK: mass 0.396271908798255 -> 0.389644381256944
- link L_KNEE_PITCH_LINK: mass 1.46957620591496 -> 1.35813128156541
- link L_PELVIS_PITCH_LINK: mass 1.38538595091799 -> 1.89700617762081
- link L_PELVIS_ROLL_LINK: mass 0.912484667273741 -> 0.92743824929528
- link L_PELVIS_YAW_LINK: mass 0.529177042283365 -> 0.530103422401833
- link L_TORQUE_SENSOR_LINK: mass 0.153697087859566 -> 0.153698480754066
- link PELVIS_LINK: mass 2.4074 -> 2.40743071856051
- link R_ANKLE_PITCH_LINK: mass 1.2402 -> 0.840739094591803
- link R_ANKLE_ROLL_LINK: mass 0.274125500097104 -> 0.274125500095123
- link R_FOOTPAD_LINK: mass 0.389644381256943 -> 0.39627
- link R_KNEE_PITCH_LINK: mass 1.4709 -> 1.35674558412184
- link R_LEG_IMU_LINK: mass 0.0368510660072014 -> 0.036851
- link R_PELVIS_PITCH_LINK: mass 1.38598662239796 -> 1.89557769383052
- link R_PELVIS_ROLL_LINK: mass 0.92744 -> 0.912484667273742
- link R_PELVIS_YAW_LINK: mass 0.530103422401833 -> 0.529177042283365
- link R_TORQUE_SENSOR_LINK: mass 0.15369584473392 -> 0.1537
- link UPPER_BODY_LINK: mass 6.0033600020323 -> 5.9955840020323
Joints:
- removed joint L_ANKLE_ROLL_LINK
- removed joint R_ANKLE_ROLL_LINK
- added joint L_ANKLE_ROLL_JOINT: type continuous, parent L_ANKLE_PITCH_LINK, child L_ANKLE_ROLL_LINK, origin xyz=-0.061 -0.049 0 rpy=0 0 0, axis 1 0 0
- added joint R_ANKLE_ROLL_JOINT: type continuous, parent R_ANKLE_PITCH_LINK, child R_ANKLE_ROLL_LINK, origin xyz=-0.061 0.049 0 rpy=0 0 0, axis -1 0 0
- joint L_ANKLE_PITCH_JOINT: limit lower=0 upper=0 effort=0 velocity=0 -> (none); origin xyz=0 0 -0.250000000000002 rpy=0 0 0 -> xyz=0 0 -0.250000000000001 rpy=0 0 0
- joint L_KNEE_PITCH_JOINT: limit lower=0 upper=0 effort=0 velocity=0 -> (none); origin xyz=0 0 -0.249999999999997 rpy=0 0 0 -> xyz=0 0 -0.25 rpy=0 0 0
- joint L_PELVIS_PITCH_JOINT: limit lower=0 upper=0 effort=0 velocity=0 -> (none); origin xyz=0.0619999999999986 -0.0489999999999418 0 rpy=0 0 0 -> xyz=0.0619999999999414 0.0489999999999982 0 rpy=0 0 0
- joint L_PELVIS_ROLL_JOINT: axis -1 0 0 -> 1 0 0; limit lower=0 upper=0 effort=0 velocity=0 -> (none); origin xyz=-0.0622500000000003 0 -0.0740000000000007 rpy=0 0 0 -> xyz=-0.06225 0 -0.0740000000000006 rpy=0 0 0
- joint L_PELVIS_YAW_JOINT: limit lower=0 upper=0 effort=0 velocity=0 -> (none); origin xyz=0 -0.07 -0.0749999999999992 rpy=0 0 0 -> xyz=0 0.07 -0.0749999999999993 rpy=0 0 0
- joint R_ANKLE_PITCH_JOINT: limit lower=0 upper=0 effort=0 velocity=0 -> (none); origin xyz=0 0 -0.250000000000001 rpy=0 0 0 -> xyz=0 0 -0.25 rpy=0 0 0
- joint R_KNEE_PITCH_JOINT: limit lower=0 upper=0 effort=0 velocity=0 -> (none)
- joint R_PELVIS_PITCH_JOINT: limit lower=0 upper=0 effort=0 velocity=0 -> (none); origin xyz=0.062 0.049 0 rpy=0 0 0 -> xyz=0.062 -0.049 0 rpy=0 0 0
- joint R_PELVIS_ROLL_JOINT: axis 1 0 0 -> -1 0 0; limit lower=0 upper=0 effort=0 velocity=0 -> (none)
- joint R_PELVIS_YAW_JOINT: limit lower=0 upper=0 effort=0 velocity=0 -> (none); origin xyz=0 0.07 -0.075 rpy=0 0 0 -> xyz=0 -0.07 -0.075 rpy=0 0 0
